File: 16 ch sample-and-hold card - single-sided.sch (EAGLE design)
At the start: 85 parts, among them IC1 MAX306CWI, IC2 TL074D, IC3 TL074D, IC4 TL074D, IC5 TL074D

Commit message: Rerouted address lines
Connections:
- net A0: now also U$1.5; no longer U$1.3
- net A2: now also U$1.3; no longer U$1.5
- net A3: now also U$1.2; no longer U$1.6
- net EN: now also U$1.6; no longer U$1.2
Other:
- moved on the sheet: U$1
Changed lines of the file:
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@@
 <part name="C43" library="resistor" deviceset="C-EU" device="C0603" value="0.1uF"/>
 <part name="C44" library="resistor" deviceset="C-EU" device="C0603" value="0.1uF"/>
-<part name="U$1" library="joakim" deviceset="MA06-1J" device="P"/>
 <part name="SV1" library="joakim" deviceset="MA20-1J" device="P"/>
 <part name="SUPPLY1" library="supply2" deviceset="DGND" device=""/>
+<part name="U$1" library="joakim" deviceset="MA06-1J" device="P"/>
 </parts>
 <sheets>
@@
 <attribute name="VALUE" x="69.596" y="121.539" size="1.778" layer="96" rot="R180"/>
 </instance>
-<instance part="U$1" gate="G$1" x="-66.04" y="-48.26"/>
 <instance part="SV1" gate="1" x="-68.58" y="5.08"/>
-<instance part="SUPPLY1" gate="G$1" x="-48.26" y="-55.88"/>
+<instance part="SUPPLY1" gate="G$1" x="-66.04" y="-40.64"/>
+<instance part="U$1" gate="G$1" x="-43.18" y="-43.18" rot="R180"/>
 </instances>
 <busses>
@@
 <wire x1="-48.26" y1="-40.64" x2="-60.96" y2="-40.64" width="0.1524" layer="91"/>
 <label x="-53.34" y="-40.64" size="1.778" layer="95"/>
-<pinref part="U$1" gate="G$1" pin="6"/>
+<pinref part="U$1" gate="G$1" pin="2"/>
 </segment>
 </net>
@@
 <wire x1="-48.26" y1="-48.26" x2="-60.96" y2="-48.26" width="0.1524" layer="91"/>
 <label x="-53.34" y="-48.26" size="1.778" layer="95"/>
-<pinref part="U$1" gate="G$1" pin="3"/>
+<pinref part="U$1" gate="G$1" pin="5"/>
 </segment>
 </net>
@@
 <wire x1="-48.26" y1="-43.18" x2="-60.96" y2="-43.18" width="0.1524" layer="91"/>
 <label x="-53.34" y="-43.18" size="1.778" layer="95"/>
-<pinref part="U$1" gate="G$1" pin="5"/>
+<pinref part="U$1" gate="G$1" pin="3"/>
 </segment>
 </net>
@@
 <wire x1="-48.26" y1="-50.8" x2="-60.96" y2="-50.8" width="0.1524" layer="91"/>
 <label x="-53.34" y="-50.8" size="1.778" layer="95"/>
-<pinref part="U$1" gate="G$1" pin="2"/>
+<pinref part="U$1" gate="G$1" pin="6"/>
 </segment>
 </net>
@@
 <net name="DGND" class="0">
 <segment>
+<wire x1="-48.26" y1="-38.1" x2="-66.04" y2="-38.1" width="0.1524" layer="91"/>
+<pinref part="SUPPLY1" gate="G$1" pin="DGND"/>
 <pinref part="U$1" gate="G$1" pin="1"/>
-<wire x1="-60.96" y1="-53.34" x2="-48.26" y2="-53.34" width="0.1524" layer="91"/>
-<pinref part="SUPPLY1" gate="G$1" pin="DGND"/>
-</segment>
-</net>
+</segment>
+</net>

Commit message: Last commit before moving multiplexer to separate repo
Other:
- note added: "Vishay DG506BE"
Changed lines of the file:
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@@
 <plain>
 <text x="-15.24" y="-27.94" size="5.08" layer="97" rot="R180">TODO: Bedre footprint for kontakt</text>
+<text x="-60.96" y="104.14" size="2.54" layer="97">Vishay
+DG506BE</text>
 </plain>
 <instances>
@@
 </schematic>
 </drawing>
+<compatibility>
+<note version="6.3" minversion="6.2.2" severity="warning">
+Since Version 6.2.2 text objects can contain more than one line,
+which will not be processed correctly with this version.
+</note>
+</compatibility>
 </eagle>
